File: eagle/Navi.brd (EAGLE design)
At the start: 26 x 18 mm, 5 parts

Commit message: first board design
Parts:
- moved JP1 3.00 mm to (26.0, 14.0)
- moved LED1 2.83 mm to (25.0, 5.00)
Routing:
- net N$17: track 26.0 -> 29.0 mm
- net N$33: track 7.10 -> 9.58 mm
- net GND: track 39.3 -> 40.3 mm
Other:
- board size 26 x 18 mm -> 28 x 18 mm
Changed lines of the file:
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@@
 <board>
 <plain>
-<wire x1="0" y1="0" x2="26" y2="0" width="0" layer="20"/>
-<wire x1="26" y1="0" x2="26" y2="18" width="0" layer="20"/>
-<wire x1="26" y1="18" x2="0" y2="18" width="0" layer="20"/>
+<wire x1="0" y1="0" x2="28" y2="0" width="0" layer="20"/>
+<wire x1="28" y1="0" x2="28" y2="18" width="0" layer="20"/>
+<wire x1="28" y1="18" x2="0" y2="18" width="0" layer="20"/>
 <wire x1="0" y1="18" x2="0" y2="0" width="0" layer="20"/>
 </plain>
@@
 </autorouter>
 <elements>
-<element name="JP1" library="pinhead" package="1X02" value="" x="23" y="14" rot="R270"/>
+<element name="JP1" library="pinhead" package="1X02" value="" x="26" y="14" rot="R270"/>
 <element name="JP2" library="pinhead" package="1X06" value="" x="3" y="9" rot="R270"/>
-<element name="LED1" library="led" package="LED3MM" value="red" x="23" y="3" rot="R90"/>
+<element name="LED1" library="led" package="LED3MM" value="red" x="25" y="5" rot="R90"/>
 <element name="R15" library="resistor" package="R1206" value="150" x="15" y="3" rot="MR180"/>
 <element name="U$2" library="0liver" package="NAVILOK-NL-631ETTL" value="NAVILOK-NL-631ETTL" x="8" y="13" rot="R270"/>
@@
 <wire x1="20" y1="3" x2="21" y2="2" width="0.6096" layer="16"/>
 <wire x1="21" y1="2" x2="22.73" y2="2" width="0.6096" layer="16"/>
-<wire x1="22.73" y1="2" x2="23" y2="1.73" width="0.6096" layer="16"/>
+<wire x1="22.73" y1="2" x2="25" y2="3.73" width="0.6096" layer="16"/>
 </signal>
 <signal name="TX">
@@
 <wire x1="3.35" y1="15" x2="3" y2="15.35" width="0.6096" layer="16"/>
 <wire x1="3" y1="15.35" x2="22.92" y2="15.35" width="0.6096" layer="16"/>
-<wire x1="22.92" y1="15.35" x2="23" y2="15.27" width="0.6096" layer="16"/>
+<wire x1="22.92" y1="15.35" x2="26" y2="15.27" width="0.6096" layer="16"/>
 </signal>
 <signal name="GND">
@@
 <contactref element="LED1" pad="K"/>
 <contactref element="JP1" pad="2"/>
-<wire x1="23" y1="12.73" x2="23" y2="4.27" width="0.6096" layer="16"/>
-<wire x1="23" y1="12.73" x2="23" y2="13" width="0.6096" layer="16"/>
-<wire x1="23" y1="13" x2="19.45" y2="13" width="0.6096" layer="16"/>
-<wire x1="19.45" y1="13" x2="18.55" y2="12.1" width="0.6096" layer="16"/>
 <wire x1="18.55" y1="12.1" x2="18.55" y2="7.7" width="0.6096" layer="16"/>
 <wire x1="18.55" y1="7.7" x2="17.7" y2="7.7" width="0.6096" layer="16"/>
@@
 <vertex x="-1" y="19"/>
 <vertex x="-1" y="-2"/>
-<vertex x="27" y="-2"/>
-<vertex x="27" y="19"/>
+<vertex x="30" y="-2"/>
+<vertex x="30" y="19"/>
 </polygon>
+<wire x1="18.55" y1="12.1" x2="25.37" y2="12.1" width="0.6096" layer="16"/>
+<wire x1="25.37" y1="12.1" x2="26" y2="12.73" width="0.6096" layer="16"/>
+<wire x1="26" y1="12.73" x2="26" y2="7.27" width="0.6096" layer="16"/>
+<wire x1="26" y1="7.27" x2="25" y2="6.27" width="0.6096" layer="16"/>
 </signal>
 <signal name="N$1">
 <polygon width="0.6096" layer="16">
 <vertex x="-3" y="20"/>
-<vertex x="29" y="20"/>
-<vertex x="29" y="-3"/>
+<vertex x="32" y="20"/>
+<vertex x="32" y="-3"/>
 <vertex x="-3" y="-3"/>
 </polygon>
